File: huxley/huxley.kicad_pcb (KiCad board)
At the start: 4 copper layers, 125 x 124 mm, 143 parts, among them J1 CT3151V1-2, J11 SMA_RF2-04A-T-00-50-G, J13 SMA_RF2-04A-T-00-50-G, J15 SMA_RF2-04A-T-00-50-G, J17 SMA_RF2-04A-T-00-50-G, J18 SMA_RF2-04A-T-00-50-G, J19 SMA_RF2-04A-T-00-50-G, J2 CT3151V1-2, J20 SMA_RF2-04A-T-00-50-G, J21 61300211121, J22 SMA_RF2-04A-T-00-50-G, J24 CT3151V1-2, J25 61300211121, J26 61300211121, J27 61300211121, J28 61300211121, J29 61300211121, J3 CT3151V1-2, J30 61300211121, J31 61300211121, J32 61300211121, J34 CT3151V1-0, J35 CT3151V1-2, J37 CT3151V1-0, J39 CT3151V1-2, J4 SMA_RF2-04A-T-00-50-G, J5 SMA_RF2-04A-T-00-50-G, J7 SMA_RF2-04A-T-00-50-G, J8 61300211121, J9 SMA_RF2-04A-T-00-50-G, U2 LM134H, U3 MAX40201FAUA+, U4 TMUX1112PWR, U5 TMUX1112PWR, U6 NVT2010PW_118

Commit message: pre edgechange
Parts:
- removed C56, C57: 1n, Capacitor_SMD:C_0603_1608Metric
- removed C58, C59: 10p, Capacitor_SMD:C_0603_1608Metric
- removed J8: 61300211121, Connector_PinHeader_2.54mm:PinHeader_1x02_P2.54mm_Vertical
- C44, C45, C46, C47, C52, C53, C54, C55, C60, C61, C62, C63: moved to B.Cu
- moved TP4 149.6 mm to (49.1, 98.5), turned to 90 degrees
- moved C55 128.5 mm to (125.8, 116.0), turned to 0 degrees
- moved C54 126.8 mm to (125.8, 117.5), turned to 0 degrees
- moved TP3 123.9 mm to (151.9, 161.1), turned to 90 degrees
- moved C60 109.5 mm to (99.5, 89.0), turned to 180 degrees
- moved C61 109.0 mm to (99.5, 90.5), turned to 180 degrees
- moved C62 108.5 mm to (99.5, 92.0), turned to 180 degrees
- moved C63 108.1 mm to (99.5, 93.5), turned to 180 degrees
- moved C52 89.0 mm to (98.5, 96.0), turned to 90 degrees
- moved C53 87.8 mm to (83.2, 119.0), turned to 180 degrees
- moved C43 82.2 mm to (80.0, 64.0), turned to -90 degrees
- moved C40 82.1 mm to (75.5, 64.0), turned to -90 degrees
- moved C42 82.0 mm to (78.5, 64.0), turned to -90 degrees
- moved C41 82.0 mm to (77.0, 64.0), turned to -90 degrees
- moved TP1 79.1 mm to (112.9, 50.6), turned to 90 degrees
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Connections:
- J6 pad 17: IBIAS_SEL4 -> IBIAS_SEL2
- J6 pad 18: IBIAS_SEL3 -> IBIAS_SEL1
- J6 pad 19: IBIAS_SEL2 -> IBIAS_SEL4
- J6 pad 20: IBIAS_SEL1 -> IBIAS_SEL3
Routing:
- net IBIAS_SEL3: track 0.00 -> 195.3 mm, vias 0 -> 3
- net IBIAS_SEL2: track 0.00 -> 193.0 mm, vias 0 -> 3
- net IBIAS_SEL1: track 0.00 -> 189.4 mm, vias 0 -> 2
- net IBIAS_SEL4: track 0.00 -> 184.4 mm, vias 0 -> 2
- net iout_dummy: track 16.8 -> 45.2 mm
- net GND: track 34.0 -> 16.6 mm, vias 36 -> 89
- net iout_dummy_amp: track 12.1 -> 17.5 mm
- net iout_dummy_amp_conn: track 13.2 -> 9.45 mm
- net vbias1: track 3.33 -> 6.07 mm
- net output_0-: track 46.2 -> 45.0 mm
- net PP_TAVDD_1V8: track 4.51 -> 3.43 mm, vias 4 -> 8
- net output_1+: track 33.0 -> 32.1 mm
- net vlvl: track 4.50 -> 3.78 mm
- net /ibias/R2_4: track 16.2 -> 16.8 mm
- net output_5+: track 35.8 -> 36.4 mm
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- added copper zone on In2.Cu, net PP_SYS_3V3
Other:
- outline, holes or cut-outs redrawn

Commit message: I can't believe it's not butter
Parts:
- C48, C49, C50, C51: moved to B.Cu
- moved C50 32.9 mm to (99.8, 138.0)
- moved C51 29.0 mm to (101.2, 138.0)
- moved C49 15.3 mm to (125.5, 129.0), turned to 0 degrees
- moved C48 13.9 mm to (125.5, 130.5), turned to 0 degrees
- moved C35 8.78 mm to (142.2, 149.0)
- moved C34 7.75 mm to (143.8, 149.0)
- moved C33 6.79 mm to (145.2, 149.0)
- moved C32 5.94 mm to (146.8, 149.0)
- moved C37 4.84 mm to (144.5, 77.0)
- moved C38 3.74 mm to (146.0, 77.0)
- moved C39 2.80 mm to (147.5, 77.0)
- moved C36 2.31 mm to (149.0, 77.0)
Routing:
- net GND: track 16.6 -> 8.01 mm, vias 89 -> 97
- net PP_VDDIO_1V8: track 6.91 -> 2.04 mm, vias 5 -> 9
- net vrbias: track 3.35 -> 0.00 mm, vias 3 -> 4
Other:
- outline, holes or cut-outs redrawn
- board text added: "I can't believe it's not butter"
- board text removed: "R1_1"
- board text removed: "R1_2"
- board text removed: "R1_3"
- board text removed: "R1_4"
- board text removed: "R2_1"
- board text removed: "R2_2"
- board text removed: "R2_3"
- board text removed: "R2_4"
- board text removed: "vbias1"
