File: huxley/huxley.kicad_sch (KiCad schematic)
At the start: 8 parts, among them J5 SMA_RF2-04A-T-00-50-G, U6 NVT2010PW_118

Commit message: removed all via-in-pad; added CLK connection to analogdiscovery signal generator
Parts:
- U1: footprint _726_Common:CPG08462 -> 0_726_footprints:CPG08462_Full
Changed lines of the file:
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@@
 			)
 		)
-		(property "Footprint" "_726_Common:CPG08462"
+		(property "Footprint" "0_726_footprints:CPG08462_Full"
 			(at 218.44 67.31 0)
 			(effects
