File: amp_board_rev2/aio.kicad_sch (KiCad schematic)
At the start: 22 parts, among them J10 SMA_RF2-04A-T-00-50-G, J11 SMA_RF2-04A-T-00-50-G, J12 SMA_RF2-04A-T-00-50-G, J13 SMA_RF2-04A-T-00-50-G, J14 SMA_RF2-04A-T-00-50-G, J15 SMA_RF2-04A-T-00-50-G, J16 SMA_RF2-04A-T-00-50-G, J17 SMA_RF2-04A-T-00-50-G, J18 SMA_RF2-04A-T-00-50-G, J19 SMA_RF2-04A-T-00-50-G, J20 SMA_RF2-04A-T-00-50-G, J21 SMA_RF2-04A-T-00-50-G, J22 SMA_RF2-04A-T-00-50-G, J23 Conn_01x06_Pin, J24 503480-3200, J25 Conn_01x06_Pin, J5 SMA_RF2-04A-T-00-50-G, J6 SMA_RF2-04A-T-00-50-G, J7 SMA_RF2-04A-T-00-50-G, J8 SMA_RF2-04A-T-00-50-G, J9 SMA_RF2-04A-T-00-50-G

Commit message: minor update
Parts:
- J23, J25: footprint Connector_PinHeader_1.00mm:PinHeader_1x06_P1.00mm_Vertical -> Connector_PinHeader_2.54mm:PinHeader_1x06_P2.54mm_Vertical
Changed lines of the file:
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@@
 			)
 		)
-		(property "Footprint" "Connector_PinHeader_1.00mm:PinHeader_1x06_P1.00mm_Vertical"
+		(property "Footprint" "Connector_PinHeader_2.54mm:PinHeader_1x06_P2.54mm_Vertical"
 			(at 251.46 53.34 0)
 			(effects
@@
 			)
 		)
-		(property "Footprint" "Connector_PinHeader_1.00mm:PinHeader_1x06_P1.00mm_Vertical"
+		(property "Footprint" "Connector_PinHeader_2.54mm:PinHeader_1x06_P2.54mm_Vertical"
 			(at 229.87 50.8 0)
 			(effects
