File: amp_board_rev2/amp0.kicad_sch (KiCad schematic)
At the start: 28 parts

Commit message: rev 3 routing
Parts:
- added C36: 0.1u, Capacitor_SMD:C_0603_1608Metric, symbol Device:C_Small
- added C37: 10u, Capacitor_SMD:C_0603_1608Metric, symbol Device:C_Small
Connections:
- net GND: now also C36.2, C37.2; no longer R24.2, R25.2
- net HV: now also C36.1, C37.1
- net output_0: now also R24.2
- net output_1: now also R25.2
Other:
- note added: "Fmax = Slew Rate / 2*pi*Vp Vp = SR/2piF = 27 V/us * 1/2*pi*1MHz = Therefore, only amplify this signal to 4V, 4x gain LPF Design: fc = (1/2pi)*sqrt(1/R3R4C2C5) R4 = R3 = 1k fc = 2e6 C2C5 = 1.56pF C5 = 1pF C2 = 1.56pF"
- note removed: "Fmax = Slew Rate / 2*pi*Vp Vp = SR/2piF = 4.29V Therefore, only amplify this signal to 4V, 4x gain LPF Design: fc = (1/2pi)*sqrt(1/R3R4C2C5) R4 = R3 = 1k fc = 2e6 C2C5 = 1.56pF C5 = 1pF C2 = 1.56pF"
- note removed: "TODO: BYPASS CAPS"
