File: amp_board_rev2/amp1.kicad_sch (KiCad schematic)
At the start: 29 parts

Commit message: rev 3 routing
Parts:
- added C34: 0.1u, Capacitor_SMD:C_0603_1608Metric, symbol Device:C_Small
- added C35: 10u, Capacitor_SMD:C_0603_1608Metric, symbol Device:C_Small
Connections:
- net GND: now also C34.2, C35.2; no longer R11.2, R24.2
- net HV: now also C34.1, C35.1
- net output_2: now also R24.2
- net output_3: now also R11.2
