File: amp_board_rev2/amp_board_rev2.kicad_pcb (KiCad board)
At the start: 4 copper layers, 148.5 x 79 mm, 110 parts, among them J1 CT3151V1-0, J10 SMA_RF2-04A-T-00-50-G, J11 SMA_RF2-04A-T-00-50-G, J12 SMA_RF2-04A-T-00-50-G, J13 SMA_RF2-04A-T-00-50-G, J14 SMA_RF2-04A-T-00-50-G, J15 SMA_RF2-04A-T-00-50-G, J16 SMA_RF2-04A-T-00-50-G, J17 SMA_RF2-04A-T-00-50-G, J18 SMA_RF2-04A-T-00-50-G, J19 SMA_RF2-04A-T-00-50-G, J2 CT3151V1-0, J20 SMA_RF2-04A-T-00-50-G, J21 SMA_RF2-04A-T-00-50-G, J22 SMA_RF2-04A-T-00-50-G, J23 Conn_01x06_Pin, J24 503480-3200, J25 Conn_01x06_Pin, J3 CT3151V1-2, J4 CT3151V1-2, J5 SMA_RF2-04A-T-00-50-G, J6 SMA_RF2-04A-T-00-50-G, J7 SMA_RF2-04A-T-00-50-G, J8 SMA_RF2-04A-T-00-50-G, J9 SMA_RF2-04A-T-00-50-G

Commit message: rev 3 routing
Routing:
- net +12V: vias 13 -> 12
Changed lines of the file:
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@@
 		(tags "OPA2211AIDDAR ")
 		(property "Reference" "U2"
-			(at 0 0 0)
+			(at -2.255 3.6325 0)
 			(unlocked yes)
 			(layer "F.SilkS")
@@
 		)
 		(fp_text user "*"
-			(at -2.87655 -3.5306 0)
-			(unlocked yes)
-			(layer "F.SilkS")
-			(effects
-				(font
-					(size 1 1)
-					(thickness 0.15)
-				)
-			)
-		)
-		(fp_text user "*"
 			(at -1.6129 -2.413 0)
 			(unlocked yes)
@@
 			)
 		)
-		(fp_text user "*"
-			(at -1.6129 -2.413 0)
+		(fp_text user "${REFERENCE}"
+			(at 0 0 0)
 			(unlocked yes)
 			(layer "F.Fab")
@@
 			)
 		)
-		(fp_text user "${REFERENCE}"
-			(at 0 0 0)
+		(fp_text user "*"
+			(at -1.6129 -2.413 0)
 			(unlocked yes)
 			(layer "F.Fab")
@@
 			(net 10 "+12V")
 			(pintype "power_in")
-			(zone_connect 2)
 		)
 		(pad "EPAD" smd rect
@@
 		(fp_line
 			(start 5 -1.68)
-			(end -3.97 -1.68)
+			(end -5 -1.68)
 			(stroke
 				(width 0.05)
@@
 		(tags "Integrated Circuit")
 		(property "Reference" "U5"
-			(at 0 0 90)
+			(at -7.9 9.75 90)
 			(layer "F.SilkS")
 			(effects
@@
 		(tags "OPA2211AIDDAR ")
 		(property "Reference" "U6"
-			(at 0 0 0)
+			(at -2.15 3.75 0)
 			(unlocked yes)
 			(layer "F.SilkS")
@@
 			)
 		)
-		(fp_text user "*"
-			(at -2.87655 -3.5306 0)
+		(fp_text user "${REFERENCE}"
+			(at 0 0 0)
 			(unlocked yes)
-			(layer "F.SilkS")
+			(layer "F.Fab")
 			(effects
 				(font
@@
 			)
 		)
-		(fp_text user "${REFERENCE}"
-			(at 0 0 0)
-			(unlocked yes)
-			(layer "F.Fab")
-			(effects
-				(font
-					(size 1 1)
-					(thickness 0.15)
-				)
-			)
-		)
 		(fp_text user "*"
 			(at -1.6129 -2.413 0)
@@
 			(net 10 "+12V")
 			(pintype "power_in")
-			(zone_connect 2)
 		)
 		(pad "EPAD" smd rect
@@
 		(fp_line
 			(start 5 -1.68)
-			(end -3.97 -1.68)
+			(end -5 -1.68)
 			(stroke
 				(width 0.05)
@@
 		(tags "CT3151V1-0 ")
 		(property "Reference" "J2"
-			(at 2.6 -6.58979 -90)
+			(at 2.7827 -7.9667 -90)
 			(unlocked yes)
 			(layer "F.SilkS")
@@
 		(fp_line
 			(start 5 -1.68)
-			(end -3.97 -1.68)
+			(end -5 -1.68)
 			(stroke
 				(width 0.05)
@@
 		(tags "Integrated Circuit")
 		(property "Reference" "U3"
-			(at 0 0 90)
+			(at -8.1 9.7 90)
 			(layer "F.SilkS")
 			(effects
@@
 		(sheetname "Analog IO")
 		(sheetfile "aio.kicad_sch")
-		(attr smd)
+		(solder_mask_margin 0.05)
+		(attr smd allow_soldermask_bridges)
 		(fp_line
 			(start -8.85 -1.575)
@@
 		(tags "Integrated Circuit")
 		(property "Reference" "U1"
-			(at 0 0 90)
+			(at -8.2 9.8 90)
 			(layer "F.SilkS")
 			(effects
@@
 		(attr through_hole)
 		(fp_arc
-			(start 0.293403 0.920976)
-			(mid -1.099243 -0.066901)
-			(end 0.412664 -0.860313)
+			(start 0.483971 1.367105)
+			(mid -0.961764 -1.211347)
+			(end 0.999999 0.999999)
 			(stroke
 				(width 0.12)
@@
 		(tags "OPA2211AIDDAR ")
 		(property "Reference" "U4"
-			(at 0 0 0)
+			(at -1.7525 3.6262 0)
 			(unlocked yes)
 			(layer "F.SilkS")
@@
 		)
 		(fp_text user "*"
-			(at -2.87655 -3.5306 0)
-			(unlocked yes)
-			(layer "F.SilkS")
-			(effects
-				(font
-					(size 1 1)
-					(thickness 0.15)
-				)
-			)
-		)
-		(fp_text user "${REFERENCE}"
-			(at 0 0 0)
+			(at -1.6129 -2.413 0)
 			(unlocked yes)
 			(layer "F.Fab")
@@
 		)
 		(fp_text user "*"
-			(at -1.6129 -2.413 0)
-			(unlocked yes)
+			(at -1.612899 -2.413 0)
 			(layer "F.Fab")
 			(effects
@@
 			)
 		)
-		(fp_text user "*"
-			(at -1.612899 -2.413 0)
+		(fp_text user "${REFERENCE}"
+			(at 0 0 0)
+			(unlocked yes)
 			(layer "F.Fab")
 			(effects
@@
 			(net 10 "+12V")
 			(pintype "power_in")
-			(zone_connect 2)
 		)
 		(pad "EPAD" smd rect
@@
 	)
 	(gr_text "OUT 5-0"
-		(at 110.1 15.5 180)
+		(at 109.75 15.1 180)
 		(layer "F.SilkS")
 		(effects
@@
 		(size 0.508)
 		(drill 0.254)
-		(layers "F.Cu" "B.Cu")
-		(free yes)
-		(net 10)
-	)
-	(via
-		(at 93.116768 58.516768)
-		(size 0.508)
-		(drill 0.254)
