File: amp_board_rev3/amp_board_rev2_backup_11.3.kicad_pro/amp0.kicad_sch (KiCad schematic)
At the start: 31 parts

Commit message: rev 3 routing
Parts:
- removed C38: 0.1u, Capacitor_SMD:C_0603_1608Metric, symbol Device:C_Small
- removed C39: 10u, Capacitor_SMD:C_0603_1608Metric, symbol Device:C_Small
- renumbered C12 to C1, C21 to C10, C24 to C13, C26 to C15, C28 to C17, C30 to C19, C33 to C22, C14 to C3, C16 to C5, C18 to C7, C20 to C9, R24 to R10, R26 to R12, R28 to R14, R32 to R18, R33 to R19, R16 to R2, R35 to R21, R37 to R23, R39 to R25, R41 to R27, R43 to R29, R17 to R3, R20 to R6, R22 to R8, U5 to U1, U6 to U2, U1 to U3, U8 to U7
Connections:
- net GND: now also R10.2, R25.2; no longer U3.25 (EPAD), U3.26, U3.27
- net input_4a renamed input_0a
- net input_4b renamed input_0b
- net input_5a renamed input_3a
- net input_5b renamed input_1b
- net output4_lv renamed output0_lv
- net output5_lv renamed output3_lv
- net output3_lv: no longer R27.2
- net output_4 renamed output_0
- net output_0: no longer R10.2
- net output_5 renamed output_1
- net output_1: no longer R25.2
- new net output1_lv: R27.2
