File: amp_board_rev3/aio.kicad_sch (KiCad schematic)
At the start: 22 parts, among them J10 SMA_RF2-04A-T-00-50-G, J11 SMA_RF2-04A-T-00-50-G, J12 SMA_RF2-04A-T-00-50-G, J13 SMA_RF2-04A-T-00-50-G, J14 SMA_RF2-04A-T-00-50-G, J15 SMA_RF2-04A-T-00-50-G, J16 SMA_RF2-04A-T-00-50-G, J17 SMA_RF2-04A-T-00-50-G, J18 SMA_RF2-04A-T-00-50-G, J19 SMA_RF2-04A-T-00-50-G, J20 SMA_RF2-04A-T-00-50-G, J21 Conn_01x06_Pin, J22 503480-3200, J23 Conn_01x06_Pin, J3 SMA_RF2-04A-T-00-50-G, J4 SMA_RF2-04A-T-00-50-G, J5 SMA_RF2-04A-T-00-50-G, J6 SMA_RF2-04A-T-00-50-G, J7 SMA_RF2-04A-T-00-50-G, J8 SMA_RF2-04A-T-00-50-G, J9 SMA_RF2-04A-T-00-50-G

Commit message: all routed
Parts:
- removed J10, J12, J14, J4, J6, J8: SMA_RF2-04A-T-00-50-G, 726_footprints:112404, symbol _PHASE:SMA_RF2-04A-T-00-50-G
Connections:
- net input_0b: now also J3.2, J3.3 (Ext), J3.4 (Ext), J3.5 (Ext)
- net input_1b: now also J5.2, J5.3 (Ext), J5.4 (Ext), J5.5 (Ext)
- net input_2b: now also J7.2, J7.3 (Ext), J7.4 (Ext), J7.5 (Ext)
- net input_3b: now also J9.2, J9.3 (Ext), J9.4 (Ext), J9.5 (Ext)
- net input_4b: now also J11.2, J11.3 (Ext), J11.4 (Ext), J11.5 (Ext)
- net input_5b: now also J13.2, J13.3 (Ext), J13.4 (Ext), J13.5 (Ext)
- net GND renamed VSS
- net VSS: no longer J11.2, J11.3 (Ext), J11.4 (Ext), J11.5 (Ext), J13.2, J13.3 (Ext), J13.4 (Ext), J13.5 (Ext), J3.2, J3.3 (Ext), J3.4 (Ext), J3.5 (Ext), J5.2, J5.3 (Ext), J5.4 (Ext), J5.5 (Ext), J7.2, J7.3 (Ext), J7.4 (Ext), J7.5 (Ext), J9.2, J9.3 (Ext), J9.4 (Ext), J9.5 (Ext)

Commit message: updates based on 11/14 meeting
Parts:
- added J10: Conn_01x02_Pin, symbol Connector:Conn_01x02_Pin
- J11, J13, J15, J16, J17, J18, J19, J20, J3, J5, J7, J9: footprint 726_footprints:112404 -> 0_726_footprints:CONN_RF2-04A-T-00-50-G_ADM
- J21, J23: footprint Connector_PinHeader_2.54mm:PinHeader_1x06_P2.54mm_Vertical -> (none)
- J22: footprint 726_footprints:Molex_5034803200 -> 5034803200
- R1: footprint 726_footprints:RESAD3322W86L1422D475 -> (none)
Connections:
- net VSS: no longer J22.33, J22.34
- net output_0: now also J10.2 (Pin_2); no longer R1.1
- new net: J10.1 (Pin_1), R1.1
- new net GND: J22.33, J22.34
