File: amp_board_rev3/amp_board_rev3.kicad_pcb (KiCad board)
At the start: 4 copper layers, 268.3 x 107.7 mm, 110 parts, among them J1 CT3151V1-0, J10 SMA_RF2-04A-T-00-50-G, J11 SMA_RF2-04A-T-00-50-G, J12 SMA_RF2-04A-T-00-50-G, J13 SMA_RF2-04A-T-00-50-G, J14 SMA_RF2-04A-T-00-50-G, J15 SMA_RF2-04A-T-00-50-G, J16 SMA_RF2-04A-T-00-50-G, J17 SMA_RF2-04A-T-00-50-G, J18 SMA_RF2-04A-T-00-50-G, J19 SMA_RF2-04A-T-00-50-G, J2 CT3151V1-2, J20 SMA_RF2-04A-T-00-50-G, J21 Conn_01x06_Pin, J22 503480-3200, J23 Conn_01x06_Pin, J3 SMA_RF2-04A-T-00-50-G, J4 SMA_RF2-04A-T-00-50-G, J5 SMA_RF2-04A-T-00-50-G, J6 SMA_RF2-04A-T-00-50-G, J7 SMA_RF2-04A-T-00-50-G, J8 SMA_RF2-04A-T-00-50-G, J9 SMA_RF2-04A-T-00-50-G, U1 SMCJ150A, U10 SMCJ150A, U13 SMCJ150A, U14 PA343, U15 PA343, U16 SMCJ150A, U2 PA343, U3 PA343, U4 SMCJ150A, U7 SMCJ150A, U8 PA343, U9 PA343

Commit message: routing complete
Parts:
- moved C14 3.01 mm to (177.4, 72.7)
- moved C26 1.91 mm to (46.9, 74.5)
- moved C10 1.87 mm to (136.0, 75.4)
- moved C22 1.12 mm to (88.2, 72.4)
- turned R3 to 0 degrees
Connections:
- net /amp_1/output_0_mv renamed /amp_1/output_2_mv
- net /amp_1/output_1_mv renamed /amp_1/output_3_mv
- net /amp_2/output_0_mv renamed /amp_2/output_4_mv
- net /amp_2/output_1_mv renamed /amp_2/output_5_mv
- R32 pad 2: /amp_2/output_0 -> output_4
- R33 pad 2: /amp_2/output_1 -> output_5
- R8 pad 2: /amp_1/output_0 -> output_2
- R9 pad 2: /amp_1/output_1 -> output_3
- U15 pad 25: Net-(U15A-EPAD) -> GND
- U15 pad 26: Net-(U15A-EPAD) -> GND
- U15 pad 27: Net-(U15A-EPAD) -> GND
- U3 pad 25: Net-(U3A-EPAD) -> GND
- U3 pad 26: Net-(U3A-EPAD) -> GND
- U3 pad 27: Net-(U3A-EPAD) -> GND
- U9 pad 25: Net-(U9A-EPAD) -> GND
- U9 pad 26: Net-(U9A-EPAD) -> GND
- U9 pad 27: Net-(U9A-EPAD) -> GND
Routing:
- net output_5: track 0.00 -> 206.1 mm, vias 0 -> 4
- net output_4: track 0.00 -> 186.8 mm, vias 0 -> 4
- net output_1: track 0.00 -> 166.7 mm, vias 0 -> 3
- net output_3: track 0.00 -> 161.6 mm, vias 0 -> 4
- net output_0: track 42.3 -> 200.3 mm, vias 0 -> 2
- net output_2: track 0.00 -> 150.2 mm, vias 0 -> 4
- net input_5b: track 0.00 -> 36.5 mm, vias 0 -> 1
- net input_3b: track 0.00 -> 35.9 mm, vias 0 -> 1
- net /amp_2/output5_mv: track 0.00 -> 35.6 mm, vias 0 -> 2
- net /amp_1/output2_mv: track 0.00 -> 35.3 mm, vias 0 -> 2
- net input_2b: track 0.00 -> 34.8 mm, vias 0 -> 1
- net /amp_2/output4_mv: track 0.00 -> 33.2 mm, vias 0 -> 2
- net /amp_1/output3_mv: track 0.00 -> 33.2 mm, vias 0 -> 2
- net /amp_0/output1_mv: track 0.00 -> 32.6 mm, vias 0 -> 2
- net input_4b: track 0.00 -> 31.4 mm, vias 0 -> 1
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Other:
- board text removed: "CHANNELS 0:1"
- board text removed: "CHANNELS 2:3"
- board text removed: "CHANNELS 4:5"
- board text removed: "LV"

Commit message: all routed
Parts:
- removed J10, J12, J14, J6, J8: SMA_RF2-04A-T-00-50-G, 726_footprints:112404
- added R38: 10, Resistor_SMD:R_0603_1608Metric, F.Cu at (38.8, 83.3)
- added R39: 100, Resistor_SMD:R_0603_1608Metric, F.Cu at (40.7, 83.3)
- added R40: 10, Resistor_SMD:R_0603_1608Metric, F.Cu at (62.9, 88.6)
- added R41: 100, Resistor_SMD:R_0603_1608Metric, F.Cu at (60.8, 88.6)
- added R42: 10, Resistor_SMD:R_0603_1608Metric, F.Cu at (116.6, 78.9)
- added R43: 100, Resistor_SMD:R_0603_1608Metric, F.Cu at (116.5, 77.0)
- added R44: 10, Resistor_SMD:R_0603_1608Metric, F.Cu at (160.3, 78.8)
- added R45: 100, Resistor_SMD:R_0603_1608Metric, F.Cu at (160.3, 77.1)
- added R46: 10, Resistor_SMD:R_0603_1608Metric, F.Cu at (204.7, 78.5)
- added R47: 100, Resistor_SMD:R_0603_1608Metric, F.Cu at (204.7, 76.6)
- added R48: 10, Resistor_SMD:R_0603_1608Metric, F.Cu at (249.6, 78.0)
- added R49: 100, Resistor_SMD:R_0603_1608Metric, F.Cu at (249.6, 75.5)
- J4: value SMA_RF2-04A-T-00-50-G -> CT3151V1-0; footprint 726_footprints:112404 -> 726_footprints:banana_plug_CT3151V1-0
- moved J4 96.6 mm to (138.3, 103.9)
- moved C16 44.0 mm to (65.2, 88.6), turned to -90 degrees
- moved C15 40.1 mm to (36.9, 83.3), turned to -90 degrees
- moved C4 17.3 mm to (160.3, 80.6), turned to 180 degrees
- moved C3 16.7 mm to (116.6, 80.8), turned to 180 degrees
- moved C27 16.1 mm to (204.7, 80.5)
- moved C28 16.0 mm to (249.6, 80.1)
Connections:
- C1 pad 2: GND -> VSS
- C10 pad 2: GND -> VSS
- C13 pad 2: GND -> VSS
- C14 pad 2: GND -> VSS
- C15 pad 2: /amp_0/input_0a_lv -> Net-(C15-Pad2)
- C16 pad 2: /amp_0/input_1a_lv -> Net-(C16-Pad2)
- C2 pad 2: GND -> VSS
- C21 pad 2: GND -> VSS
- C22 pad 2: GND -> VSS
- C25 pad 2: GND -> VSS
- C26 pad 2: GND -> VSS
- C27 pad 2: /amp_2/input_4a_lv -> Net-(C27-Pad2)
- C28 pad 2: /amp_2/input_5a_lv -> Net-(C28-Pad2)
- C3 pad 2: /amp_1/input_2a_lv -> Net-(C3-Pad2)
- C33 pad 2: GND -> VSS
- C34 pad 2: GND -> VSS
- C37 pad 2: GND -> VSS
- C38 pad 2: GND -> VSS
- C4 pad 2: /amp_1/input_3a_lv -> Net-(C4-Pad2)
- C9 pad 2: GND -> VSS
- J1 pad 1: GND -> VSS
- J1 pad 2: GND -> VSS
- J1 pad 3: GND -> VSS
- J1 pad 4: GND -> VSS
- J11 pad 2: GND -> input_4b
- J11 pad 3: GND -> input_4b
- J11 pad 4: GND -> input_4b
- J11 pad 5: GND -> input_4b
- J13 pad 2: GND -> input_5b
- J13 pad 3: GND -> input_5b
- J13 pad 4: GND -> input_5b
- J13 pad 5: GND -> input_5b
- J15 pad 2: GND -> VSS
- J15 pad 3: GND -> VSS
- J15 pad 4: GND -> VSS
- J15 pad 5: GND -> VSS
- J16 pad 2: GND -> VSS
- J16 pad 3: GND -> VSS
- J16 pad 4: GND -> VSS
- J16 pad 5: GND -> VSS
- J17 pad 2: GND -> VSS
- J17 pad 3: GND -> VSS
- J17 pad 4: GND -> VSS
- J17 pad 5: GND -> VSS
- J18 pad 2: GND -> VSS
- J18 pad 3: GND -> VSS
- J18 pad 4: GND -> VSS
- J18 pad 5: GND -> VSS
- J19 pad 2: GND -> VSS
- J19 pad 3: GND -> VSS
- J19 pad 4: GND -> VSS
- J19 pad 5: GND -> VSS
- J20 pad 2: GND -> VSS
- J20 pad 3: GND -> VSS
- J20 pad 4: GND -> VSS
- J20 pad 5: GND -> VSS
- J21 pad 1: GND -> VSS
- J21 pad 2: GND -> VSS
- J21 pad 3: GND -> VSS
- J21 pad 4: GND -> VSS
- J21 pad 5: GND -> VSS
- J21 pad 6: GND -> VSS
- J22 pad 33: GND -> VSS
- J22 pad 34: GND -> VSS
- J3 pad 2: GND -> input_0b
- J3 pad 3: GND -> input_0b
- J3 pad 4: GND -> input_0b
- J3 pad 5: GND -> input_0b
- J4 pad 1: input_0b -> GND
- J5 pad 2: GND -> input_1b
- J5 pad 3: GND -> input_1b
- J5 pad 4: GND -> input_1b
- J5 pad 5: GND -> input_1b
- J7 pad 2: GND -> input_2b
- J7 pad 3: GND -> input_2b
- J7 pad 4: GND -> input_2b
- J7 pad 5: GND -> input_2b
- J9 pad 2: GND -> input_3b
- J9 pad 3: GND -> input_3b
- J9 pad 4: GND -> input_3b
- J9 pad 5: GND -> input_3b
- R1 pad 2: GND -> VSS
- U1 pad 2: GND -> VSS
- U10 pad 2: GND -> VSS
- U13 pad 2: GND -> VSS
- U14 pad 12: GND -> VSS
- U14 pad 24: GND -> VSS
- U14 pad 25: GND -> VSS
- U14 pad 26: GND -> VSS
- U14 pad 27: GND -> VSS
- U14 pad 9: GND -> VSS
- U15 pad 12: GND -> VSS
- U15 pad 24: GND -> VSS
- U15 pad 25: GND -> VSS
- U15 pad 26: GND -> VSS
- U15 pad 27: GND -> VSS
- U15 pad 9: GND -> VSS
- U16 pad 2: GND -> VSS
- U2 pad 12: GND -> VSS
- U2 pad 24: GND -> VSS
- U2 pad 25: GND -> VSS
- U2 pad 26: GND -> VSS
- U2 pad 27: GND -> VSS
- U2 pad 9: GND -> VSS
- U3 pad 12: GND -> VSS
- U3 pad 24: GND -> VSS
- U3 pad 25: GND -> VSS
- U3 pad 26: GND -> VSS
- U3 pad 27: GND -> VSS
- U3 pad 9: GND -> VSS
- U4 pad 2: GND -> VSS
- U7 pad 2: GND -> VSS
- U8 pad 12: GND -> VSS
- U8 pad 24: GND -> VSS
- U8 pad 25: GND -> VSS
- U8 pad 26: GND -> VSS
- U8 pad 27: GND -> VSS
- U8 pad 9: GND -> VSS
- U9 pad 12: GND -> VSS
- U9 pad 24: GND -> VSS
- U9 pad 25: GND -> VSS
- U9 pad 26: GND -> VSS
- U9 pad 27: GND -> VSS
- U9 pad 9: GND -> VSS
Routing:
- net GND: track 0.00 -> 474.4 mm, vias 110 -> 6
- net /amp_0/input_1a_lv: track 4.80 -> 97.0 mm
- net input_1a: track 98.8 -> 7.66 mm
- net input_0a: track 55.5 -> 11.3 mm
- net /amp_0/input_0a_lv: track 4.27 -> 43.5 mm
- net input_1b: track 116.8 -> 93.0 mm
- net input_3a: track 25.3 -> 7.17 mm
- net /amp_2/input_5a_lv: track 6.07 -> 23.3 mm
- net /amp_1/input_3a_lv: track 5.14 -> 22.1 mm
- net input_4a: track 24.1 -> 7.22 mm
- net input_2a: track 23.7 -> 7.06 mm
- net /amp_1/input_2a_lv: track 5.03 -> 21.4 mm
- net input_5a: track 24.1 -> 7.84 mm
- net /amp_2/input_4a_lv: track 5.52 -> 19.1 mm
- net input_5b: track 36.5 -> 25.3 mm
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- added copper zone on B.Cu, net VSS
- added copper zone on F.Cu, net VSS
- added copper zone on In1.Cu, net VSS
- added copper zone on B.Cu, net input_0b
- added copper zone on B.Cu, net input_1b
- added copper zone on B.Cu, net input_2b
- added copper zone on B.Cu, net input_3b
- added copper zone on B.Cu, net input_4b
- added copper zone on B.Cu, net input_5b
- removed copper zone on F.Cu, net GND
- removed copper zone on In1.Cu, net GND
- removed copper zone on In2.Cu, net Net-(U3B--IN_B)
Other:
- board text added: "VSS"

Commit message: ground reference pcb placement
Parts:
- added C39: 0.1u, 500V, Capacitor_SMD:C_1812_4532Metric, F.Cu at (270.5, 98.8)
- added C40: EEU-EB2G100, 726_footprints:EEU-EB2G100, F.Cu at (275.8, 107.7)
- added C41: 0.1u, 500V, Capacitor_SMD:C_1812_4532Metric, F.Cu at (145.3, 50.6)
- added C42: EEU-EB2G100, 726_footprints:EEU-EB2G100, F.Cu at (126.7, 75.4)
- added C43: 0.1u, 500V, Capacitor_SMD:C_1812_4532Metric, F.Cu at (186.3, 49.6)
- added C44: EEU-EB2G100, 726_footprints:EEU-EB2G100, F.Cu at (169.7, 73.8)
- added C45: 0.1u, 500V, Capacitor_SMD:C_1812_4532Metric, F.Cu at (56.6, 49.7)
- added C46: EEU-EB2G100, 726_footprints:EEU-EB2G100, F.Cu at (36.3, 74.5)
- added C47: 0.1u, 500V, Capacitor_SMD:C_1812_4532Metric, F.Cu at (97.0, 48.1)
- added C48: EEU-EB2G100, 726_footprints:EEU-EB2G100, F.Cu at (77.2, 72.6)
- added C49: 0.1u, 500V, Capacitor_SMD:C_1812_4532Metric, F.Cu at (234.4, 50.7)
- added C50: EEU-EB2G100, 726_footprints:EEU-EB2G100, F.Cu at (216.5, 75.4)
- added C51: 0.1u, 500V, Capacitor_SMD:C_1812_4532Metric, F.Cu at (275.7, 48.9)
- added C52: EEU-EB2G100, 726_footprints:EEU-EB2G100, F.Cu at (259.8, 73.5)
- added J6: CT3151V1-0, 726_footprints:banana_plug_CT3151V1-0, F.Cu at (260.1, 103.3)
- added J8: CT3151V1-0, 726_footprints:banana_plug_CT3151V1-0, F.Cu at (154.4, 103.9)
- added U11: SMCJ150A, 726_footprints:SMCJ150A-13-F, F.Cu at (48.4, 47.7)
- added U12: SMCJ150A, 726_footprints:SMCJ150A-13-F, F.Cu at (88.8, 46.2)
- added U17: SMCJ150A, 726_footprints:SMCJ150A-13-F, F.Cu at (225.8, 48.7)
- added U18: SMCJ150A, 726_footprints:SMCJ150A-13-F, F.Cu at (267.3, 47.0)
- added U5: SMCJ150A, 726_footprints:SMCJ150A-13-F, F.Cu at (137.2, 48.7)
- added U6: SMCJ150A, 726_footprints:SMCJ150A-13-F, F.Cu at (178.1, 47.5)
- R12, R13, R18, R19, R24, R25, R30, R31, R36, R37, R6, R7: value 100 -> 70.7
- moved C38 4.00 mm to (270.8, 73.4)
- moved C14 3.17 mm to (180.4, 73.9)
- moved C34 2.27 mm to (227.6, 74.9)
- moved C10 1.38 mm to (137.4, 75.2)
Connections:
- C1 pad 2: VSS -> GND
- C10 pad 2: VSS -> GND
- C13 pad 2: VSS -> GND
- C14 pad 2: VSS -> GND
- C2 pad 2: VSS -> GND
- C21 pad 2: VSS -> GND
- C22 pad 2: VSS -> GND
- C25 pad 2: VSS -> GND
- C26 pad 2: VSS -> GND
- C33 pad 2: VSS -> GND
- C34 pad 2: VSS -> GND
- C37 pad 2: VSS -> GND
- C38 pad 2: VSS -> GND
- C9 pad 2: VSS -> GND
- U1 pad 2: VSS -> GND
- U10 pad 2: VSS -> GND
- U13 pad 2: VSS -> GND
- U14 pad 10: Net-(U14A-NC_1) -> unconnected-(U14A-NC_1-Pad2)
- U14 pad 11: Net-(U14A-NC_1) -> unconnected-(U14A-NC_1-Pad2)
- U14 pad 14: Net-(U14A-NC_1) -> unconnected-(U14A-NC_1-Pad2)
- U14 pad 19: Net-(U14A-NC_1) -> unconnected-(U14A-NC_1-Pad2)
- U14 pad 2: Net-(U14A-NC_1) -> unconnected-(U14A-NC_1-Pad2)
- U14 pad 22: Net-(U14A-NC_1) -> unconnected-(U14A-NC_1-Pad2)
- U14 pad 23: Net-(U14A-NC_1) -> unconnected-(U14A-NC_1-Pad2)
- U14 pad 7: Net-(U14A-NC_1) -> unconnected-(U14A-NC_1-Pad2)
- U14 pad 9: VSS -> GND
- U15 pad 10: Net-(U15A-NC_1) -> unconnected-(U15A-NC_1-Pad2)
- U15 pad 11: Net-(U15A-NC_1) -> unconnected-(U15A-NC_1-Pad2)
- U15 pad 14: Net-(U15A-NC_1) -> unconnected-(U15A-NC_1-Pad2)
- U15 pad 19: Net-(U15A-NC_1) -> unconnected-(U15A-NC_1-Pad2)
- U15 pad 2: Net-(U15A-NC_1) -> unconnected-(U15A-NC_1-Pad2)
- U15 pad 22: Net-(U15A-NC_1) -> unconnected-(U15A-NC_1-Pad2)
- U15 pad 23: Net-(U15A-NC_1) -> unconnected-(U15A-NC_1-Pad2)
- U15 pad 7: Net-(U15A-NC_1) -> unconnected-(U15A-NC_1-Pad2)
- U15 pad 9: VSS -> GND
- U16 pad 2: VSS -> GND
- U2 pad 10: Net-(U2A-NC_1) -> unconnected-(U2A-NC_1-Pad2)
- U2 pad 11: Net-(U2A-NC_1) -> unconnected-(U2A-NC_1-Pad2)
- U2 pad 14: Net-(U2A-NC_1) -> unconnected-(U2A-NC_1-Pad2)
- U2 pad 19: Net-(U2A-NC_1) -> unconnected-(U2A-NC_1-Pad2)
- U2 pad 2: Net-(U2A-NC_1) -> unconnected-(U2A-NC_1-Pad2)
- U2 pad 22: Net-(U2A-NC_1) -> unconnected-(U2A-NC_1-Pad2)
- U2 pad 23: Net-(U2A-NC_1) -> unconnected-(U2A-NC_1-Pad2)
- U2 pad 7: Net-(U2A-NC_1) -> unconnected-(U2A-NC_1-Pad2)
- U2 pad 9: VSS -> GND
- U3 pad 10: Net-(U3A-NC_1) -> unconnected-(U3A-NC_1-Pad2)
- U3 pad 11: Net-(U3A-NC_1) -> unconnected-(U3A-NC_1-Pad2)
- U3 pad 14: Net-(U3A-NC_1) -> unconnected-(U3A-NC_1-Pad2)
- U3 pad 19: Net-(U3A-NC_1) -> unconnected-(U3A-NC_1-Pad2)
- U3 pad 2: Net-(U3A-NC_1) -> unconnected-(U3A-NC_1-Pad2)
- U3 pad 22: Net-(U3A-NC_1) -> unconnected-(U3A-NC_1-Pad2)
- U3 pad 23: Net-(U3A-NC_1) -> unconnected-(U3A-NC_1-Pad2)
- U3 pad 7: Net-(U3A-NC_1) -> unconnected-(U3A-NC_1-Pad2)
- U3 pad 9: VSS -> GND
- U4 pad 2: VSS -> GND
- U7 pad 2: VSS -> GND
- U8 pad 10: Net-(U8A-NC_1) -> unconnected-(U8A-NC_1-Pad2)
- U8 pad 11: Net-(U8A-NC_1) -> unconnected-(U8A-NC_1-Pad2)
- U8 pad 14: Net-(U8A-NC_1) -> unconnected-(U8A-NC_1-Pad2)
- U8 pad 19: Net-(U8A-NC_1) -> unconnected-(U8A-NC_1-Pad2)
- U8 pad 2: Net-(U8A-NC_1) -> unconnected-(U8A-NC_1-Pad2)
- U8 pad 22: Net-(U8A-NC_1) -> unconnected-(U8A-NC_1-Pad2)
- U8 pad 23: Net-(U8A-NC_1) -> unconnected-(U8A-NC_1-Pad2)
- U8 pad 7: Net-(U8A-NC_1) -> unconnected-(U8A-NC_1-Pad2)
- U8 pad 9: VSS -> GND
- U9 pad 10: Net-(U9A-NC_1) -> unconnected-(U9A-NC_1-Pad2)
- U9 pad 11: Net-(U9A-NC_1) -> unconnected-(U9A-NC_1-Pad2)
- U9 pad 14: Net-(U9A-NC_1) -> unconnected-(U9A-NC_1-Pad2)
- U9 pad 19: Net-(U9A-NC_1) -> unconnected-(U9A-NC_1-Pad2)
- U9 pad 2: Net-(U9A-NC_1) -> unconnected-(U9A-NC_1-Pad2)
- U9 pad 22: Net-(U9A-NC_1) -> unconnected-(U9A-NC_1-Pad2)
- U9 pad 23: Net-(U9A-NC_1) -> unconnected-(U9A-NC_1-Pad2)
- U9 pad 7: Net-(U9A-NC_1) -> unconnected-(U9A-NC_1-Pad2)
- U9 pad 9: VSS -> GND
Routing:
- net VSS: vias 110 -> 113
- added copper zone on F.Cu, net GND
- removed copper zone on B.Cu, net VSS
Other:
- board text added: "In_0"
- board text added: "In_1"
- board text added: "In_2"
- board text added: "In_3"
- board text added: "In_4"
- board text added: "In_5"
- board text removed: "In_0a"
- board text removed: "In_0b"
- board text removed: "In_1a"
- board text removed: "In_1b"
- board text removed: "In_2a"
- board text removed: "In_2b"
- board text removed: "In_3a"
- board text removed: "In_3b"
- board text removed: "In_4a"
- board text removed: "In_4b"
- board text removed: "In_5a"
- board text removed: "In_5b"

Commit message: added polygons for ground reference
Parts:
- moved C10 2.05 mm to (139.4, 75.4)
- moved C34 0.55 mm to (227.9, 75.4)
Routing:
- net VSS: vias 113 -> 161
- net HV: vias 72 -> 150

Commit message: updates based on 11/14 meeting
Parts:
- added J10: Conn_01x02_Pin, Connector_PinHeader_2.54mm:PinHeader_1x02_P2.54mm_Vertical, F.Cu at (185.7, 22.1)
- C11, C12, C19, C20, C31, C32: value 0.24pF, 500V -> 0.75pF, 250V; footprint Capacitor_SMD:C_0402_1005Metric -> Capacitor_SMD:C_0805_2012Metric
- C23, C24, C35, C36, C7, C8: value 0.24pF, 500V -> 0.2pF, 250V; footprint Capacitor_SMD:C_0402_1005Metric -> Capacitor_SMD:C_0805_2012Metric
- moved C18 41.2 mm to (66.5, 59.5)
- moved C20 41.2 mm to (91.2, 58.2)
- moved C25 41.2 mm to (79.5, 42.1)
- moved C26 41.2 mm to (88.0, 73.3)
- moved C45 41.2 mm to (97.8, 48.4)
- moved C46 41.2 mm to (77.4, 73.3)
- moved R25 41.2 mm to (92.2, 55.4)
- moved U10 41.2 mm to (77.6, 50.0)
- moved U9 41.2 mm to (81.3, 57.8)
- moved C24 41.2 mm to (71.2, 54.2)
- moved R15 41.2 mm to (92.2, 61.6)
- moved R17 41.2 mm to (70.3, 59.6)
- moved R19 41.2 mm to (70.3, 56.8)
- moved R21 41.2 mm to (70.2, 51.7)
- moved R23 41.2 mm to (92.3, 53.2)
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Connections:
- J22 pad 33: VSS -> GND
- J22 pad 34: VSS -> GND
- R1 pad 1: output_0 -> Net-(J10-Pin_1)
Routing:
- net /amp_0/input_1a_lv: track 97.0 -> 35.4 mm
- net GND: track 474.4 -> 422.7 mm, vias 6 -> 11
- net output_5: track 206.1 -> 230.8 mm, vias 4 -> 3
- net output_1: track 166.7 -> 188.4 mm
- net /amp_0/input_0a_lv: track 43.5 -> 22.2 mm
- net output_3: track 161.6 -> 181.6 mm
- net output_4: track 186.8 -> 205.5 mm
- net output_0: track 200.3 -> 210.2 mm
- net output_2: track 150.2 -> 142.4 mm
- net Net-(J10-Pin_1): track 0.00 -> 6.76 mm
- net input_0a: track 11.3 -> 9.61 mm
