File: amp_board_rev3/amp_board_rev3.kicad_pcb (KiCad board)
At the start: 4 copper layers, 268.3 x 107.7 mm, 140 parts, among them J1 CT3151V1-0, J10 Conn_01x02_Pin, J11 SMA_RF2-04A-T-00-50-G, J13 SMA_RF2-04A-T-00-50-G, J15 SMA_RF2-04A-T-00-50-G, J16 SMA_RF2-04A-T-00-50-G, J17 SMA_RF2-04A-T-00-50-G, J18 SMA_RF2-04A-T-00-50-G, J19 SMA_RF2-04A-T-00-50-G, J2 CT3151V1-2, J20 SMA_RF2-04A-T-00-50-G, J21 Conn_01x06_Pin, J22 503480-3200, J23 Conn_01x06_Pin, J3 SMA_RF2-04A-T-00-50-G, J4 CT3151V1-0, J5 SMA_RF2-04A-T-00-50-G, J6 CT3151V1-0, J7 SMA_RF2-04A-T-00-50-G, J8 CT3151V1-0, J9 SMA_RF2-04A-T-00-50-G, U1 SMCJ150A, U10 SMCJ150A, U11 SMCJ150A, U12 SMCJ150A, U13 SMCJ150A, U14 PA343, U15 PA343, U16 SMCJ150A, U17 SMCJ150A, U18 SMCJ150A, U2 PA343, U3 PA343, U4 SMCJ150A, U5 SMCJ150A, U6 SMCJ150A, U7 SMCJ150A, U8 PA343, U9 PA343

Commit message: detailed adjustments
Parts:
- C11, C12: value 0.75pF, 250V -> 0.2pF, 250V
- C7, C8: value 0.2pF, 250V -> 0.75pF, 250V
- moved R9 1.32 mm to (159.7, 52.6)
- moved R20 1.00 mm to (29.4, 52.6)
- moved R8 0.97 mm to (118.4, 53.6)
- moved C21 0.96 mm to (38.1, 43.9)
- moved C33 0.92 mm to (215.9, 43.2)
- moved U13 0.82 mm to (214.9, 51.2)
- moved C20 0.81 mm to (91.9, 58.4)
- moved C31 0.71 mm to (229.1, 60.2)
- moved C11 0.70 mm to (118.6, 56.6)
- moved C23 0.69 mm to (30.0, 55.6)
- moved C7 0.69 mm to (140.7, 60.5)
- moved R21 0.64 mm to (70.2, 51.1)
- moved C19 0.63 mm to (50.8, 60.2)
- moved C35 0.63 mm to (207.3, 57.4)
- moved C12 0.59 mm to (160.0, 55.9)
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Connections:
- U14 pad 10: unconnected-(U14A-NC_1-Pad2) -> unconnected-(U14A-NC-Pad10)
- U14 pad 11: unconnected-(U14A-NC_1-Pad2) -> unconnected-(U14A-NC-Pad11)
- U14 pad 14: unconnected-(U14A-NC_1-Pad2) -> unconnected-(U14A-NC-Pad14)
- U14 pad 19: unconnected-(U14A-NC_1-Pad2) -> unconnected-(U14B-NC-Pad19)
- U14 pad 2: unconnected-(U14A-NC_1-Pad2) -> unconnected-(U14B-NC-Pad2)
- U14 pad 22: unconnected-(U14A-NC_1-Pad2) -> unconnected-(U14B-NC-Pad22)
- U14 pad 23: unconnected-(U14A-NC_1-Pad2) -> unconnected-(U14B-NC-Pad23)
- U14 pad 7: unconnected-(U14A-NC_1-Pad2) -> unconnected-(U14A-NC-Pad7)
- U15 pad 10: unconnected-(U15A-NC_1-Pad2) -> unconnected-(U15A-NC-Pad10)
- U15 pad 11: unconnected-(U15A-NC_1-Pad2) -> unconnected-(U15A-NC-Pad11)
- U15 pad 14: unconnected-(U15A-NC_1-Pad2) -> unconnected-(U15A-NC-Pad14)
- U15 pad 19: unconnected-(U15A-NC_1-Pad2) -> unconnected-(U15B-NC-Pad19)
- U15 pad 2: unconnected-(U15A-NC_1-Pad2) -> unconnected-(U15B-NC-Pad2)
- U15 pad 22: unconnected-(U15A-NC_1-Pad2) -> unconnected-(U15B-NC-Pad22)
- U15 pad 23: unconnected-(U15A-NC_1-Pad2) -> unconnected-(U15B-NC-Pad23)
- U15 pad 7: unconnected-(U15A-NC_1-Pad2) -> unconnected-(U15A-NC-Pad7)
- U2 pad 10: unconnected-(U2A-NC_1-Pad2) -> unconnected-(U2A-NC-Pad10)
- U2 pad 11: unconnected-(U2A-NC_1-Pad2) -> unconnected-(U2A-NC-Pad11)
- U2 pad 14: unconnected-(U2A-NC_1-Pad2) -> unconnected-(U2A-NC-Pad14)
- U2 pad 19: unconnected-(U2A-NC_1-Pad2) -> unconnected-(U2B-NC-Pad19)
- U2 pad 2: unconnected-(U2A-NC_1-Pad2) -> unconnected-(U2B-NC-Pad2)
- U2 pad 22: unconnected-(U2A-NC_1-Pad2) -> unconnected-(U2B-NC-Pad22)
- U2 pad 23: unconnected-(U2A-NC_1-Pad2) -> unconnected-(U2B-NC-Pad23)
- U2 pad 7: unconnected-(U2A-NC_1-Pad2) -> unconnected-(U2A-NC-Pad7)
- U3 pad 10: unconnected-(U3A-NC_1-Pad2) -> unconnected-(U3A-NC-Pad10)
- U3 pad 11: unconnected-(U3A-NC_1-Pad2) -> unconnected-(U3A-NC-Pad11)
- U3 pad 14: unconnected-(U3A-NC_1-Pad2) -> unconnected-(U3A-NC-Pad14)
- U3 pad 19: unconnected-(U3A-NC_1-Pad2) -> unconnected-(U3B-NC-Pad19)
- U3 pad 2: unconnected-(U3A-NC_1-Pad2) -> unconnected-(U3B-NC-Pad2)
- U3 pad 22: unconnected-(U3A-NC_1-Pad2) -> unconnected-(U3B-NC-Pad22)
- U3 pad 23: unconnected-(U3A-NC_1-Pad2) -> unconnected-(U3B-NC-Pad23)
- U3 pad 7: unconnected-(U3A-NC_1-Pad2) -> unconnected-(U3A-NC-Pad7)
- U8 pad 10: unconnected-(U8A-NC_1-Pad2) -> unconnected-(U8A-NC-Pad10)
- U8 pad 11: unconnected-(U8A-NC_1-Pad2) -> unconnected-(U8A-NC-Pad11)
- U8 pad 14: unconnected-(U8A-NC_1-Pad2) -> unconnected-(U8A-NC-Pad14)
- U8 pad 19: unconnected-(U8A-NC_1-Pad2) -> unconnected-(U8B-NC-Pad19)
- U8 pad 2: unconnected-(U8A-NC_1-Pad2) -> unconnected-(U8B-NC-Pad2)
- U8 pad 22: unconnected-(U8A-NC_1-Pad2) -> unconnected-(U8B-NC-Pad22)
- U8 pad 23: unconnected-(U8A-NC_1-Pad2) -> unconnected-(U8B-NC-Pad23)
- U8 pad 7: unconnected-(U8A-NC_1-Pad2) -> unconnected-(U8A-NC-Pad7)
- U9 pad 10: unconnected-(U9A-NC_1-Pad2) -> unconnected-(U9A-NC-Pad10)
- U9 pad 11: unconnected-(U9A-NC_1-Pad2) -> unconnected-(U9A-NC-Pad11)
- U9 pad 14: unconnected-(U9A-NC_1-Pad2) -> unconnected-(U9A-NC-Pad14)
- U9 pad 19: unconnected-(U9A-NC_1-Pad2) -> unconnected-(U9B-NC-Pad19)
- U9 pad 2: unconnected-(U9A-NC_1-Pad2) -> unconnected-(U9B-NC-Pad2)
- U9 pad 22: unconnected-(U9A-NC_1-Pad2) -> unconnected-(U9B-NC-Pad22)
- U9 pad 23: unconnected-(U9A-NC_1-Pad2) -> unconnected-(U9B-NC-Pad23)
- U9 pad 7: unconnected-(U9A-NC_1-Pad2) -> unconnected-(U9A-NC-Pad7)
Routing:
- net GND: track 422.7 -> 19.5 mm, vias 11 -> 6
- net input_1b: track 93.0 -> 28.1 mm
- net output_2: track 142.4 -> 172.2 mm, vias 4 -> 5
- net input_0b: track 49.5 -> 24.6 mm
- net output_0: track 210.2 -> 228.5 mm, vias 2 -> 3
- net output_4: track 205.5 -> 213.0 mm, vias 4 -> 5
- net output_1: track 188.4 -> 182.5 mm, vias 3 -> 4
- net Net-(U14B-CC_B_1): track 0.00 -> 5.35 mm
- net Net-(U14B-CC_B_2): track 0.00 -> 4.78 mm
- net output_5: track 230.8 -> 235.3 mm, vias 3 -> 4
- net output_3: track 181.6 -> 184.5 mm, vias 4 -> 5
- net /amp_2/output4_mv: track 33.2 -> 36.0 mm, vias 2 -> 3
- net /amp_2/input_5a_lv: track 23.3 -> 21.4 mm
- net /amp_1/input_2a_lv: track 21.4 -> 20.5 mm
- net Net-(U2B-CC_B_1): track 4.56 -> 5.49 mm
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Other:
- board text added: "Jumper to Test Load"
- board text added: "OUT 0-31"
- board text removed: "OUT 31-0"
