File: amp_board_rev3/amp_board_rev3.kicad_pcb (KiCad board)
At the start: 4 copper layers, 268.3 x 107.7 mm, 140 parts, among them J1 CT3151V1-0, J10 Conn_01x02_Pin, J11 SMA_RF2-04A-T-00-50-G, J13 SMA_RF2-04A-T-00-50-G, J15 SMA_RF2-04A-T-00-50-G, J16 SMA_RF2-04A-T-00-50-G, J17 SMA_RF2-04A-T-00-50-G, J18 SMA_RF2-04A-T-00-50-G, J19 SMA_RF2-04A-T-00-50-G, J2 CT3151V1-2, J20 SMA_RF2-04A-T-00-50-G, J21 Conn_01x06_Pin, J22 503480-3200, J23 Conn_01x06_Pin, J3 SMA_RF2-04A-T-00-50-G, J4 CT3151V1-0, J5 SMA_RF2-04A-T-00-50-G, J6 CT3151V1-0, J7 SMA_RF2-04A-T-00-50-G, J8 CT3151V1-0, J9 SMA_RF2-04A-T-00-50-G, U1 SMCJ150A, U10 SMCJ150A, U11 SMCJ150A, U12 SMCJ150A, U13 SMCJ150A, U14 PA343, U15 PA343, U16 SMCJ150A, U17 SMCJ150A, U18 SMCJ150A, U2 PA343, U3 PA343, U4 SMCJ150A, U5 SMCJ150A, U6 SMCJ150A, U7 SMCJ150A, U8 PA343, U9 PA343

Commit message: final fabrication generated
Parts:
- added J12: Conn_01x06_Pin, Connector_PinHeader_2.54mm:PinHeader_1x06_P2.54mm_Vertical, F.Cu at (127.6, 32.6)
- moved C38 1.10 mm to (269.8, 73.9)
- moved C52 0.92 mm to (258.9, 73.9)
- moved C22 0.55 mm to (47.2, 74.1)
- moved C46 0.35 mm to (77.1, 73.3)
- moved J21 0.35 mm to (127.6, 27.3)
- moved C26 0.27 mm to (88.3, 73.3)
- moved C48 0.23 mm to (36.6, 74.1)
