File: amp_board_rev3/amp0_c1.kicad_sch (KiCad schematic)
At the start: 38 parts, among them U1 SMCJ150A, U10 SMCJ150A, U2 PA343, U3 PA343, U5 SMCJ150A, U6 SMCJ150A

Commit message: final fabrication generated
Parts:
- R22, R23, R4, R42, R44, R5: value 10 -> 100
- R24, R25, R6, R7: value 70.7 -> 707
- R43, R45: value 100 -> 707
