File: amp_board_rev3_backup_11.15/amp0.kicad_sch (KiCad schematic)
At the start: 38 parts, among them U1 SMCJ150A, U10 SMCJ150A, U2 PA343, U3 PA343, U5 SMCJ150A, U6 SMCJ150A

Commit message: detailed adjustments
Parts:
- removed C41, C43: 0.1u, 500V, Capacitor_SMD:C_1812_4532Metric, symbol Device:C_Small
- removed C42, C44: EEU-EB2G100, 726_footprints:EEU-EB2G100, symbol _PHASE:EEU-EB2G100
- removed R42, R44: 10, symbol Device:R_US
- removed R43, R45: 100, symbol Device:R_US
- removed unit 2 of U2
- removed unit 2 of U3
- removed U5, U6: SMCJ150A, 726_footprints:SMCJ150A-13-F, symbol _PHASE:SMCJ150A-13-F
- added C45, C47: 0.1u, 500V, symbol Device:C_Small
- added C46, C48: EEU-EB2G100, CAPPRD500W65D1000H2200, symbol _PHASE:EEU-EB2G100
- added R38, R40: 10, symbol Device:R_US
- added R39, R41: 100, symbol Device:R_US
- added U11, U12: SMCJ150A, 726_footprints:SMCJ150A-13-F, symbol _PHASE:SMCJ150A-13-F
- added unit 2 of U8
- added unit 2 of U9
- C15, C16, C17, C18: footprint Capacitor_SMD:C_0603_1608Metric -> (none)
- C19: renamed from C7; footprint Capacitor_SMD:C_0805_2012Metric -> (none)
- C20: renamed from C8; footprint Capacitor_SMD:C_0805_2012Metric -> (none)
- C21: renamed from C9; footprint Capacitor_SMD:C_1812_4532Metric -> (none)
- C22: renamed from C10; footprint 726_footprints:EEU-EB2G100 -> CAPPRD500W65D1000H2200
- C23, C24: footprint Capacitor_SMD:C_0805_2012Metric -> (none)
- C25: footprint Capacitor_SMD:C_1812_4532Metric -> (none)
- C26: renamed from C14; footprint 726_footprints:EEU-EB2G100 -> CAPPRD500W65D1000H2200
- U8: renamed from U2; footprint 726_footprints:PA341DF -> (none)
- U9: renamed from U3; footprint 726_footprints:PA341DF -> (none)
- renumbered R2 to R14, R3 to R15, R4 to R16, R5 to R17, R6 to R18, R7 to R19, U1 to U7
Connections:
- net GND: now also C45.1, C46.1 (+), C47.1, C48.1 (+), R39.1, R41.1, U11.1 (K), U12.1 (K), U8.9 (+IN_B), U9.9 (+IN_B)
- net HV: now also U8.13, U9.13
- net VSS: now also C45.2, C46.2 (-), C47.2, C48.2 (-), U11.2 (A), U12.2 (A), U8.12, U9.12
- net at R21.1: now also U9.15 (CL_B)
- net at C16.2: now also R40.2
- net at R20.1: now also U8.15 (CL_B)
- net at C23.1: now also U8.16 (CC_B_1)
- net at C23.2: now also U8.17 (CC_B_2)
- net at R22.1, R24.2: now also U8.8 (-IN_B)
- net at R23.1, R25.2: now also U9.8 (-IN_B)
- net at C24.1: now also U9.16 (CC_B_1)
- net at C24.2: now also U9.17 (CC_B_2)
- net at C15.2: now also R38.2
- net input_2a renamed input_0a
- net input_2a_lv renamed input_0a_lv
- net input_0a_lv: now also R38.1, R39.2
- net input_2b renamed input_0b
- net input_2b_lv renamed input_0b_lv
- net input_3a renamed input_1a
- net input_3a_lv renamed input_1a_lv
- net input_1a_lv: now also R40.1, R41.2
- net input_3b renamed input_1b
- net input_3b_lv renamed input_1b_lv
- net output2_mv renamed output0_mv
- net output3_mv renamed output1_mv
- net output_2 renamed output_0
- net output_0: now also U8.18 (OUT_B)
- net output_2_mv renamed output_0_mv
- net output_3 renamed output_1
- net output_1: now also U9.18 (OUT_B)
- net output_3_mv renamed output_1_mv
- no-connect marks 18 -> 2
