File: amp_board_rev3_backup_11.15/amp0_c1.kicad_sch (KiCad schematic)
At the start: 38 parts, among them U1 SMCJ150A, U10 SMCJ150A, U2 PA343, U3 PA343, U5 SMCJ150A, U6 SMCJ150A

Commit message: detailed adjustments
Parts:
- removed unit 2 of U2
- removed unit 2 of U3
- added unit 2 of U2
- added U9: PA343, 726_footprints:PA341DF, symbol _PHASE:PA343_2Units
- C10, C14, C42, C44: footprint 726_footprints:EEU-EB2G100 -> CAPPRD500W65D1000H2200
- C15, C16, C17, C18: footprint Capacitor_SMD:C_0603_1608Metric -> (none)
- C23, C24, C7, C8: footprint Capacitor_SMD:C_0805_2012Metric -> (none)
- C25, C41, C43, C9: footprint Capacitor_SMD:C_1812_4532Metric -> (none)
- U2, U3: footprint 726_footprints:PA341DF -> (none)
Connections:
- net GND: now also U2.9 (+IN_B), U9.9 (+IN_B)
- net HV: now also U2.13, U9.13
- net VSS: now also U2.12, U9.12
- net output_2: now also U2.18 (OUT_B)
- net output_3: now also U9.18 (OUT_B)
- net at R21.1: now also U9.15 (CL_B)
- net at R20.1: now also U2.15 (CL_B)
- net at C23.1: now also U2.16 (CC_B_1)
- net at C23.2: now also U2.17 (CC_B_2)
- net at R22.1, R24.2: now also U2.8 (-IN_B)
- net at R23.1, R25.2: now also U9.8 (-IN_B)
- net at C24.1: now also U9.16 (CC_B_1)
- net at C24.2: now also U9.17 (CC_B_2)
- no-connect marks 18 -> 2
