File: amp_board_rev3_backup_11.15/amp0_c2.kicad_sch (KiCad schematic)
At the start: 38 parts, among them U1 SMCJ150A, U10 SMCJ150A, U2 PA343, U3 PA343, U5 SMCJ150A, U6 SMCJ150A

Commit message: detailed adjustments
Parts:
- removed C41, C43: 0.1u, 500V, Capacitor_SMD:C_1812_4532Metric, symbol Device:C_Small
- removed C42, C44: EEU-EB2G100, 726_footprints:EEU-EB2G100, symbol _PHASE:EEU-EB2G100
- removed R42, R44: 10, symbol Device:R_US
- removed R43, R45: 100, symbol Device:R_US
- removed unit 2 of U2
- removed unit 2 of U3
- removed U5, U6: SMCJ150A, 726_footprints:SMCJ150A-13-F, symbol _PHASE:SMCJ150A-13-F
- added C49, C51: 0.1u, 500V, symbol Device:C_Small
- added C50, C52: EEU-EB2G100, CAPPRD500W65D1000H2200, symbol _PHASE:EEU-EB2G100
- added R46, R48: 10, symbol Device:R_US
- added R47, R49: 100, symbol Device:R_US
- added unit 2 of U14
- added U17, U18: SMCJ150A, 726_footprints:SMCJ150A-13-F, symbol _PHASE:SMCJ150A-13-F
- added U9: PA343, 726_footprints:PA341DF, symbol _PHASE:PA343_2Units
- C15, C16, C17, C18: footprint Capacitor_SMD:C_0603_1608Metric -> (none)
- C23, C24: footprint Capacitor_SMD:C_0805_2012Metric -> (none)
- C25: footprint Capacitor_SMD:C_1812_4532Metric -> (none)
- C31: renamed from C7; footprint Capacitor_SMD:C_0805_2012Metric -> (none)
- C32: renamed from C8; footprint Capacitor_SMD:C_0805_2012Metric -> (none)
- C33: renamed from C9; footprint Capacitor_SMD:C_1812_4532Metric -> (none)
- C34: renamed from C10; footprint 726_footprints:EEU-EB2G100 -> CAPPRD500W65D1000H2200
- C38: renamed from C14; footprint 726_footprints:EEU-EB2G100 -> CAPPRD500W65D1000H2200
- U14: renamed from U2; footprint 726_footprints:PA341DF -> (none)
- U15: renamed from U3; footprint 726_footprints:PA341DF -> (none)
- renumbered R2 to R26, R3 to R27, R4 to R28, R5 to R29, R6 to R30, R7 to R31, U1 to U13
Connections:
- net GND: now also C49.1, C50.1 (+), C51.1, C52.1 (+), R47.1, R49.1, U14.9 (+IN_B), U17.1 (K), U18.1 (K), U9.9 (+IN_B)
- net HV: now also U14.13, U9.13
- net VSS: now also C49.2, C50.2 (-), C51.2, C52.2 (-), U14.12, U17.2 (A), U18.2 (A), U9.12
- net at R21.1: now also U9.15 (CL_B)
- net at C16.2: now also R48.2
- net at R20.1: now also U14.15 (CL_B)
- net at C23.1: now also U14.16 (CC_B_1)
- net at C23.2: now also U14.17 (CC_B_2)
- net at R22.1, R24.2: now also U14.8 (-IN_B)
- net at R23.1, R25.2: now also U9.8 (-IN_B)
- net at C24.1: now also U9.16 (CC_B_1)
- net at C24.2: now also U9.17 (CC_B_2)
- net at C15.2: now also R46.2
- net input_2a renamed input_4a
- net input_2a_lv renamed input_4a_lv
- net input_4a_lv: now also R46.1, R47.2
- net input_2b renamed input_4b
- net input_2b_lv renamed input_4b_lv
- net input_3a renamed input_5a
- net input_3a_lv renamed input_5a_lv
- net input_5a_lv: now also R48.1, R49.2
- net input_3b renamed input_5b
- net input_3b_lv renamed input_5b_lv
- net output2_mv renamed output4_mv
- net output3_mv renamed output5_mv
- net output_2 renamed output_4
- net output_4: now also U14.18 (OUT_B)
- net output_2_mv renamed output_4_mv
- net output_3 renamed output_5
- net output_5: now also U9.18 (OUT_B)
- net output_3_mv renamed output_5_mv
- no-connect marks 18 -> 2
