File: amp_board_rev3_backup_11.15/boardPower.kicad_sch (KiCad schematic)
At the start: 9 parts, among them J1 CT3151V1-0, J2 CT3151V1-2, J4 CT3151V1-0, J6 CT3151V1-0, J8 CT3151V1-0

Commit message: detailed adjustments
Parts:
- C1, C39: footprint Capacitor_SMD:C_1812_4532Metric -> (none)
- C2, C40: footprint 726_footprints:EEU-EB2G100 -> CAPPRD500W65D1000H2200
Changed lines of the file:
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@@
 			)
 		)
-		(property "Footprint" "726_footprints:EEU-EB2G100"
+		(property "Footprint" "CAPPRD500W65D1000H2200"
 			(at -7.29 67.31 0)
 			(effects
@@
 			)
 		)
-		(property "Footprint" "Capacitor_SMD:C_1812_4532Metric"
+		(property "Footprint" ""
 			(at 134.62 74.93 0)
 			(effects
@@
 			)
 		)
-		(property "Footprint" "Capacitor_SMD:C_1812_4532Metric"
+		(property "Footprint" ""
 			(at 67.31 71.12 0)
 			(effects
@@
 			)
 		)
-		(property "Footprint" "726_footprints:EEU-EB2G100"
+		(property "Footprint" "CAPPRD500W65D1000H2200"
 			(at 60.02 78.74 0)
 			(effects
